File: eps_version_0.4.0.brd (EAGLE design)
At the start: 90.2 x 95.5 mm, 186 parts, among them J1 2PIN_HEADER, J2 2PIN_HEADER, J3 2PIN_HEADER, J4 2PIN_HEADER, J5 2PIN_HEADER, J6 2PIN_HEADER, J7 CONN_2X5_127, J8 USB-C, M1 A03400, U1 MP2639A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

Commit message: synced files
Parts:
- C2: value 1uF -> 0
- C60: value 0.1uF -> C61
- R15: value 1K -> 0
- R16: value 1K -> DNP
Connections:
- net LX: no longer C5.1
- net U1_SW: now also C5.1
