File: eps_version_0.4.0.sch (EAGLE design)
At the start: 186 parts, among them J1 2PIN_HEADER, J2 2PIN_HEADER, J3 2PIN_HEADER, J4 2PIN_HEADER, J5 2PIN_HEADER, J6 2PIN_HEADER, J7 CONN_2X5_127, J8 USB-C, M1 A03400, U1 MP2639A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

Commit message: synced files
Parts:
- C2: value 1uF -> 0
- C60: value 0.1uF -> C61
- R15: value 1K -> 0
- R16: value 1K -> DNP
Connections:
- net LX: no longer C5.1
- net U1_SW: now also C5.1
Changed lines of the file:
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@@
 <part name="U4" library="HSFL_Main_Library" deviceset="LT8609A" device=""/>
 <part name="U5" library="HSFL_Main_Library" deviceset="LT8609A" device=""/>
-<part name="C60" library="HSFL_Main_Library" deviceset="CAP" device="0805" value="0.1uF"/>
+<part name="C60" library="HSFL_Main_Library" deviceset="CAP" device="0805" value="C61"/>
 <part name="C61" library="HSFL_Main_Library" deviceset="CAP" device="0805" value="0.1uF"/>
 <part name="C62" library="HSFL_Main_Library" deviceset="CAP" device="0805" value="0.1uF"/>
@@
 <part name="LED5" library="DSD_Passive_Library" deviceset="LED_0805" device=""/>
 <part name="LED6" library="DSD_Passive_Library" deviceset="LED_0805" device=""/>
-<part name="C2" library="DSD_Passive_Library" deviceset="CAP" device="0603-CAP" value="1uF"/>
+<part name="C2" library="DSD_Passive_Library" deviceset="CAP" device="0603-CAP" value="0"/>
 <part name="R7" library="DSD_Passive_Library" deviceset="RESISTOR" device="0603-RES" value="2K"/>
 <part name="R8" library="DSD_Passive_Library" deviceset="RESISTOR" device="0603-RES" value="2K"/>
@@
 <part name="R10" library="DSD_Passive_Library" deviceset="RESISTOR" device="0603-RES" value="10K"/>
 <part name="D8" library="DSD_Passive_Library" deviceset="DIODE" device="-SOD123" value="1N5819HW"/>
-<part name="R15" library="DSD_Passive_Library" deviceset="RESISTOR" device="0603-RES" value="1K"/>
-<part name="R16" library="DSD_Passive_Library" deviceset="RESISTOR" device="0603-RES" value="1K"/>
+<part name="R15" library="DSD_Passive_Library" deviceset="RESISTOR" device="0603-RES" value="0"/>
+<part name="R16" library="DSD_Passive_Library" deviceset="RESISTOR" device="0603-RES" value="DNP"/>
 <part name="R17" library="DSD_Passive_Library" deviceset="RESISTOR" device="0603-RES" value="100"/>
 <part name="R18" library="DSD_Passive_Library" deviceset="RESISTOR" device="0603-RES" value="1K"/>
@@
 <pinref part="L1" gate="A" pin="1"/>
 <wire x1="101.6" y1="114.3" x2="99.06" y2="114.3" width="0.1524" layer="91"/>
-<pinref part="C5" gate="G$1" pin="1"/>
-<wire x1="99.06" y1="114.3" x2="88.9" y2="114.3" width="0.1524" layer="91"/>
-<wire x1="88.9" y1="111.76" x2="88.9" y2="114.3" width="0.1524" layer="91"/>
 <wire x1="99.06" y1="124.46" x2="99.06" y2="114.3" width="0.1524" layer="91"/>
 <junction x="99.06" y="114.3"/>
@@
 <pinref part="U1" gate="A" pin="SW"/>
 <wire x1="116.84" y1="114.3" x2="119.38" y2="114.3" width="0.1524" layer="91"/>
-</segment>
-</net>
+<pinref part="C5" gate="G$1" pin="1"/>
+<wire x1="88.9" y1="111.76" x2="88.9" y2="116.84" width="0.1524" layer="91"/>
+<wire x1="88.9" y1="116.84" x2="116.84" y2="116.84" width="0.1524" layer="91"/>
+<wire x1="116.84" y1="116.84" x2="116.84" y2="114.3" width="0.1524" layer="91"/>
+<junction x="116.84" y="114.3"/>
+</segment>
+</net>
